Commit message: Update to last brainCo Updates

File: urdf/revo2_left_hand.urdf (robot description, URDF)
Before this commit: robot brainco_revo2_lefthand_urdf, 22 links, 21 joints
Joints:
- joint left_thumb_distal_joint: mimic joint=left_thumb_proximal_joint multiplier=1 offset=0 -> joint=left_thumb_proximal_joint multiplier=0.691851 offset=0.0395854; origin xyz=0 -0.052 0 rpy=0 0 0 -> xyz=0 -0.052 0 rpy=0.10472 0 0
- joint left_thumb_proximal_joint: origin xyz=0 -0.014227 0 rpy=-0.17488 0.23736 -0.16787 -> xyz=0 -0.014227 0 rpy=-0.33153 0.23736 -0.16787

File: urdf/revo2_right_hand.urdf (robot description, URDF)
Before this commit: robot brainco_revo2_righthand_urdf, 22 links, 21 joints
Joints:
- joint right_thumb_distal_joint: mimic joint=right_thumb_proximal_joint multiplier=1 offset=0 -> joint=right_thumb_proximal_joint multiplier=0.691851 offset=0.0395854; origin xyz=0 0.052 0 rpy=0 0 0 -> xyz=0 0.052 0 rpy=-0.10472 0 0
- joint right_thumb_proximal_joint: origin xyz=0 0.014227 0 rpy=0.17488 0.23736 0.16787 -> xyz=0 0.014227 0 rpy=0.33153 0.23736 0.16787
